File: LT3483/LT3483.kicad_pcb (KiCad board)
At the start: 2 copper layers, 19.8 x 50.5 mm, 20 parts, among them J1 J1, J2 J2, U1 LT3483

Commit message: upravy, pred vyrobou, opraven problem s maskou
Parts:
- C8: value (none) -> 1uF/50V
- J1: value J1 -> Conn_02x03_Odd_Even
- J2: value J2 -> Conn_02x04_Odd_Even
- R1: value 39R -> 39.2R
- R2: value 3.2M -> 3.24M
- gave numbers to parts that had none: 4
Connections:
- MH1 pad 1: Net-(MH1-Pad1) -> (no net)
- MH2 pad 1: Net-(MH2-Pad1) -> (no net)
- MH3 pad 1: Net-(MH3-Pad1) -> (no net)
- MH4 pad 1: Net-(MH4-Pad1) -> (no net)

Commit message: Oprava_1.01
Parts:
- moved MH1 0.25 mm to (172.7, 132.1)
- moved MH2 0.25 mm to (182.9, 132.1)
Other:
- board size 19.8 x 50.5 mm -> 19.8 x 50.3 mm
Changed lines of the file:
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@@
-(kicad_pcb (version 20171130) (host pcbnew "(6.0.0-rc1-dev-205-gc0615c5ef)")
+(kicad_pcb (version 20171130) (host pcbnew "(5.0.0)")
   (general
     (thickness 1.6)
@@
     (zone_45_only no)
     (trace_min 0.2)
+    (segment_width 0.2)
+    (edge_width 0.15)
     (via_size 0.8)
     (via_drill 0.4)
@@
     (uvia_min_size 0.2)
     (uvia_min_drill 0.1)
-    (edge_width 0.15)
-    (segment_width 0.2)
     (pcb_text_width 0.3)
     (pcb_text_size 1.5 1.5)
@@
   )
   (module MountingHole:MountingHole_3mm_Pad locked (layer F.Cu)
-    (at 172.72 132.334 90)
+    (at 172.72 132.08 90)
     (descr "Mounting Hole 3mm")
     (tags "mounting hole 3mm")
     (attr virtual)
-    (fp_text reference MH1 (at 0 -4 90) (layer F.SilkS)
+    (fp_text reference MH1 (at 0 -4 90) (layer F.SilkS) hide
       (effects (font (size 1 1) (thickness 0.15)))
     )
@@
     (pad 1 thru_hole circle (at 0 0 90) (size 6 6) (drill 3) (layers *.Cu *.Mask))
   )
-  (module MountingHole:MountingHole_3mm_Pad locked (layer F.Cu)
-    (at 182.88 132.334 90)
+  (module MountingHole:MountingHole_3mm_Pad (layer F.Cu)
+    (at 182.88 132.08 90)
     (descr "Mounting Hole 3mm")
     (tags "mounting hole 3mm")
     (attr virtual)
-    (fp_text reference MH2 (at 0 -4 90) (layer F.SilkS)
+    (fp_text reference MH2 (at 0 -4 90) (layer F.SilkS) hide
       (effects (font (size 1 1) (thickness 0.15)))
     )
@@
     (tags "mounting hole 3mm")
     (attr virtual)
-    (fp_text reference MH3 (at 0 -4 90) (layer F.SilkS)
+    (fp_text reference MH3 (at 0 -4 90) (layer F.SilkS) hide
       (effects (font (size 1 1) (thickness 0.15)))
     )
@@
     (tags "mounting hole 3mm")
     (attr virtual)
-    (fp_text reference MH4 (at 0 -4 90) (layer F.SilkS)
+    (fp_text reference MH4 (at 0 -4 90) (layer F.SilkS) hide
       (effects (font (size 1 1) (thickness 0.15)))
     )
@@
     (descr "Through hole straight pin header, 2x03, 2.54mm pitch, double rows")
     (tags "Through hole pin header THT 2x03 2.54mm double row")
-    (fp_text reference J1 (at 1.27 -3.048 90) (layer F.SilkS)
+    (fp_text reference J1 (at 1.27 -3.048 90) (layer F.SilkS) hide
       (effects (font (size 1 1) (thickness 0.15)))
     )
@@
     (descr "Through hole straight pin header, 2x04, 2.54mm pitch, double rows")
     (tags "Through hole pin header THT 2x04 2.54mm double row")
-    (fp_text reference J2 (at 1.27 -3.048 90) (layer F.SilkS)
+    (fp_text reference J2 (at 1.27 -3.048 90) (layer F.SilkS) hide
       (effects (font (size 1 1) (thickness 0.15)))
     )
@@
     )
   )
+  (gr_line (start 187.706 129.286) (end 187.706 136.906) (layer Edge.Cuts) (width 0.15))
+  (gr_line (start 167.894 129.286) (end 167.894 136.906) (layer Edge.Cuts) (width 0.15))
+  (gr_line (start 167.894 136.906) (end 187.706 136.906) (layer Edge.Cuts) (width 0.15))
   (gr_line (start 176.276 108.204) (end 176.276 106.426) (layer F.Fab) (width 0.2))
   (gr_line (start 178.562 108.204) (end 176.276 108.204) (layer F.Fab) (width 0.2))
   (gr_line (start 178.562 106.426) (end 178.562 108.204) (layer F.Fab) (width 0.2))
   (gr_line (start 176.276 106.426) (end 178.562 106.426) (layer F.Fab) (width 0.2))
-  (gr_line (start 167.894 129.286) (end 167.894 137.16) (layer Edge.Cuts) (width 0.15))
-  (gr_line (start 187.706 129.286) (end 187.706 137.16) (layer Edge.Cuts) (width 0.15))
   (gr_line (start 167.894 129.286) (end 167.894 86.614) (layer Edge.Cuts) (width 0.15))
-  (gr_line (start 187.706 137.16) (end 167.894 137.16) (layer Edge.Cuts) (width 0.15))
   (gr_line (start 187.706 86.614) (end 187.706 129.286) (layer Edge.Cuts) (width 0.15))
   (gr_line (start 167.894 86.614) (end 187.706 86.614) (layer Edge.Cuts) (width 0.15))
@@
     (polygon
       (pts
-        (xy 168.656 87.376) (xy 186.944 87.376) (xy 186.944 136.398) (xy 168.656 136.398)
+        (xy 186.944 136.144) (xy 186.944 87.376) (xy 168.656 87.376) (xy 168.656 136.144)
       )
     )
@@
     (polygon
       (pts
-        (xy 168.656 87.376) (xy 186.944 87.376) (xy 186.944 136.398) (xy 168.656 136.398)
+        (xy 186.944 136.144) (xy 168.656 136.144) (xy 168.656 87.376) (xy 186.944 87.376)
       )
     )

Commit message: generovani vyrobnich dat a oprava maskovani soucastky
Parts:
- L1: footprint digikey-footprints:LQH2MCN100K02L -> Mlab_L:LQH2MCN100K02L
Changed lines of the file:
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@@
-(kicad_pcb (version 20171130) (host pcbnew "(5.0.0)")
+(kicad_pcb (version 20171130) (host pcbnew "(6.0.0-rc1-dev-205-gc0615c5ef)")
   (general
     (thickness 1.6)
@@
     (zone_45_only no)
     (trace_min 0.2)
-    (segment_width 0.2)
-    (edge_width 0.15)
     (via_size 0.8)
     (via_drill 0.4)
@@
     (uvia_min_size 0.2)
     (uvia_min_drill 0.1)
+    (edge_width 0.15)
+    (segment_width 0.2)
     (pcb_text_width 0.3)
     (pcb_text_size 1.5 1.5)
@@
     (add_net "Net-(D1-Pad2)")
   )
-  (module digikey-footprints:LQH2MCN100K02L (layer F.Cu)
+  (module Mlab_L:LQH2MCN100K02L (layer F.Cu)
     (at 177.419 107.315 180)
     (descr LQH2M)
@@
       (effects (font (size 1.27 1.27) (thickness 0.254)))
     )
+    (fp_circle (center -1.551 -0.018) (end -1.551 -0.007) (layer F.SilkS) (width 0.2))
+    (fp_line (start 1 0.8) (end -1 0.8) (layer F.SilkS) (width 0.2))
+    (fp_line (start -1 -0.8) (end 1 -0.8) (layer F.SilkS) (width 0.2))
+    (fp_line (start -1 0.8) (end -1 -0.8) (layer Dwgs.User) (width 0.2))
+    (fp_line (start 1 0.8) (end -1 0.8) (layer Dwgs.User) (width 0.2))
+    (fp_line (start 1 -0.8) (end 1 0.8) (layer Dwgs.User) (width 0.2))
     (fp_line (start -1 -0.8) (end 1 -0.8) (layer Dwgs.User) (width 0.2))
-    (fp_line (start 1 -0.8) (end 1 0.8) (layer Dwgs.User) (width 0.2))
-    (fp_line (start 1 0.8) (end -1 0.8) (layer Dwgs.User) (width 0.2))
-    (fp_line (start -1 0.8) (end -1 -0.8) (layer Dwgs.User) (width 0.2))
-    (fp_line (start -1 -0.8) (end 1 -0.8) (layer F.SilkS) (width 0.2))
-    (fp_line (start 1 0.8) (end -1 0.8) (layer F.SilkS) (width 0.2))
-    (fp_circle (center -1.551 -0.018) (end -1.551 -0.007) (layer F.SilkS) (width 0.2))
-    (pad 1 smd rect (at -0.85 0 180) (size 0.9 1) (layers F.Cu F.Paste)
+    (pad 2 smd rect (at 0.85 0 180) (size 0.9 1) (layers F.Cu F.Paste F.Mask)
+      (net 4 "Net-(C3-Pad1)"))
+    (pad 1 smd rect (at -0.85 0 180) (size 0.9 1) (layers F.Cu F.Paste F.Mask)
       (net 2 "Net-(C1-Pad2)"))
-    (pad 2 smd rect (at 0.85 0 180) (size 0.9 1) (layers F.Cu F.Paste)
-      (net 4 "Net-(C3-Pad1)"))
   )
   (module Diode_SMD:D_SOD-123 (layer F.Cu)
