File: LT3483/LT3483.sch (KiCad schematic (older format))
At the start: 15 parts, among them J1 Conn_02x03_Odd_Even, J2 Conn_02x04_Odd_Even, U1 LT3483

Commit message: Update
Parts:
- added C2: 100nF/30V, Capacitor_SMD:C_0805_2012Metric, symbol Device:C
- added C6, C7: 100nF, Capacitor_SMD:C_0805_2012Metric, symbol Device:C
- added C8: 1uF/50V, Capacitor_SMD:C_0805_2012Metric, symbol Device:C
- added R3: 100R, Resistor_SMD:R_0805_2012Metric, symbol Device:R
- C1: value 4.7uF/10V -> 4.7uF/30V
- J1: footprint Connector_PinHeader_2.00mm:PinHeader_2x03_P2.00mm_Vertical -> Connector_PinHeader_2.54mm:PinHeader_2x03_P2.54mm_Vertical
- J2: footprint Connector_PinHeader_2.00mm:PinHeader_2x04_P2.00mm_Vertical -> Connector_PinHeader_2.54mm:PinHeader_2x04_P2.54mm_Vertical
- renumbered C2 to C3, C3 to C4, C4 to C5
Connections:
- wire segments 71 -> 84

Commit message: New components
Parts:
- R2: value 3.2M -> 3.24M
Changed lines of the file:
@@
 P 6300 3600
 F 0 "R2" H 6230 3554 50  0000 R CNN
-F 1 "3.2M" H 6230 3645 50  0000 R CNN
+F 1 "3.24M" H 6230 3645 50  0000 R CNN
 F 2 "Resistor_SMD:R_0805_2012Metric" V 6230 3600 50  0001 C CNN
 F 3 "~" H 6300 3600 50  0001 C CNN

Commit message: new component
Parts:
- R1: value 39R -> 39.2R
Changed lines of the file:
@@
 P 6300 3100
 F 0 "R1" H 6370 3146 50  0000 L CNN
-F 1 "39R" H 6370 3055 50  0000 L CNN
+F 1 "39.2R" H 6370 3055 50  0000 L CNN
 F 2 "Resistor_SMD:R_0805_2012Metric" V 6230 3100 50  0001 C CNN
 F 3 "~" H 6300 3100 50  0001 C CNN
