File: TPS65133/TPS65133_2.kicad_pcb (KiCad board)
At the start: 2 copper layers, 19.8 x 40.1 mm, 14 parts, among them IC1 TPS65133DPDR, J1 Conn_02x03_Odd_Even, J2 Conn_02x03_Odd_Even, J3 Conn_02x03_Odd_Even

Commit message: TPS65133
Parts:
- removed C1: 100nF, Capacitor_SMD:C_0805_2012Metric
- added ?: 100nF, Capacitor_SMD:C_0805_2012Metric, F.Cu at (115.1, 75.6)
- renumbered J2 to +5V, J3 to -5V, J1 to 2.9-5V, MH3 to ?, MH4 to ?, C2 to ?, C3 to ?, C4 to ?, IC1 to ?, L1 to ?, L2 to ?, MH1 to ?, MH2 to ?
Changed lines of the file:
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@@
     (38 B.Mask user)
     (39 F.Mask user)
-    (40 Dwgs.User user hide)
+    (40 Dwgs.User user)
     (41 Cmts.User user)
     (42 Eco1.User user)
@@
     (tags capacitor)
     (attr smd)
-    (fp_text reference C1 (at 0.173907 0.219262) (layer F.SilkS)
+    (fp_text reference "" (at 2.548321 1.400848 90) (layer F.SilkS)
       (effects (font (size 1 1) (thickness 0.15)))
     )
@@
     (tags capacitor)
     (attr smd)
-    (fp_text reference C2 (at 0 -1.65 270) (layer F.SilkS)
+    (fp_text reference "" (at 0 -1.65 270) (layer F.SilkS)
       (effects (font (size 1 1) (thickness 0.15)))
     )
@@
     (tags capacitor)
     (attr smd)
-    (fp_text reference C3 (at -0.034738 -0.095407 270) (layer F.SilkS)
+    (fp_text reference "" (at -0.034738 -0.095407 270) (layer F.SilkS)
       (effects (font (size 1 1) (thickness 0.15)))
     )
@@
     (tags capacitor)
     (attr smd)
-    (fp_text reference C4 (at 0 0 90) (layer F.SilkS)
+    (fp_text reference "" (at 0 0 90) (layer F.SilkS)
       (effects (font (size 1 1) (thickness 0.15)))
     )
@@
     (tags "Integrated Circuit")
     (attr smd)
-    (fp_text reference IC1 (at 0 0 90) (layer F.SilkS)
+    (fp_text reference "" (at 0 0 90) (layer F.SilkS)
       (effects (font (size 1.27 1.27) (thickness 0.254)))
     )
@@
     (descr "Through hole straight pin header, 2x03, 2.00mm pitch, double rows")
     (tags "Through hole pin header THT 2x03 2.00mm double row")
-    (fp_text reference J1 (at 1 -2.06 180) (layer F.SilkS)
+    (fp_text reference 2.9-5V (at 0.596414 -3.302 180) (layer F.SilkS)
       (effects (font (size 1 1) (thickness 0.15)))
     )
@@
     (descr "Through hole straight pin header, 2x03, 2.00mm pitch, double rows")
     (tags "Through hole pin header THT 2x03 2.00mm double row")
-    (fp_text reference J2 (at 1 -2.06 90) (layer F.SilkS)
+    (fp_text reference +5V (at 0.927586 -3.136414 90) (layer F.SilkS)
       (effects (font (size 1 1) (thickness 0.15)))
     )
@@
     (descr "Through hole straight pin header, 2x03, 2.00mm pitch, double rows")
     (tags "Through hole pin header THT 2x03 2.00mm double row")
-    (fp_text reference J3 (at 1 -2.06 90) (layer F.SilkS)
+    (fp_text reference -5V (at 1.27 -2.794 90) (layer F.SilkS)
       (effects (font (size 1 1) (thickness 0.15)))
     )
@@
     (tags Inductor)
     (attr smd)
-    (fp_text reference L1 (at 0 0.219262) (layer F.SilkS)
+    (fp_text reference "" (at 0 0.219262) (layer F.SilkS)
       (effects (font (size 1.27 1.27) (thickness 0.254)))
     )
@@
     (tags Inductor)
     (attr smd)
-    (fp_text reference L2 (at 0 -0.034738) (layer F.SilkS)
+    (fp_text reference "" (at 0 -0.034738) (layer F.SilkS)
       (effects (font (size 1.27 1.27) (thickness 0.254)))
     )
@@
     (tags "mounting hole 3mm")
     (attr virtual)
-    (fp_text reference MH1 (at 0 -4) (layer F.SilkS)
+    (fp_text reference "" (at 0 -4) (layer F.SilkS)
       (effects (font (size 1 1) (thickness 0.15)))
     )
@@
     (tags "mounting hole 3mm")
     (attr virtual)
-    (fp_text reference MH2 (at 0 -4) (layer F.SilkS)
+    (fp_text reference "" (at 0 -4) (layer F.SilkS)
       (effects (font (size 1 1) (thickness 0.15)))
     )
@@
     (tags "mounting hole 3mm")
     (attr virtual)
-    (fp_text reference MH3 (at 0 -4) (layer F.SilkS)
+    (fp_text reference "" (at 0 -4) (layer F.SilkS)
       (effects (font (size 1 1) (thickness 0.15)))
     )
@@
     (tags "mounting hole 3mm")
     (attr virtual)
-    (fp_text reference MH4 (at 0 -4) (layer F.SilkS)
-      (effects (font (size 1 1) (thickness 0.15)))
-    )
+    (fp_text reference "" (at 0 -4) (layer F.SilkS)
+      (effects (font (size 1 1) (thickness 0.15)))
+    )

Commit message: Update
Parts:
- removed the -5V at (120.4, 70.9)
- removed the ? at (120.7, 74.2)
- removed the ? at (119.6, 78.9)
- removed the ? at (116.7, 72.8)
- added -5V: , Connector_PinHeader_2.54mm:PinHeader_2x03_P2.54mm_Vertical, F.Cu at (116.8, 72.4)
- added C4: GRM21BR71A106KE5, Capacitor_SMD:C_0805_2012Metric, F.Cu at (121.0, 75.4)
- added C5: GRM21BR71E104KA01, Capacitor_SMD:C_0805_2012Metric, F.Cu at (121.7, 90.0)
- added C6: GRM21BR71E104KA01, Capacitor_SMD:C_0805_2012Metric, F.Cu at (121.0, 77.5)
- added L2: 1239AS-H-4R7M=P2, SamacSys_Parts:1239AS-H-4R7M=P2, F.Cu at (116.0, 77.2)
- added U1: TPS65133DPDR, SamacSys_Parts:SON45P300X300X80-13N-D, F.Cu at (119.8, 84.0)
- +3.3V: renamed from 2.9-5V; value Conn_02x03_Odd_Even -> (none); footprint Connector_PinHeader_2.00mm:PinHeader_2x03_P2.00mm_Vertical -> Connector_PinHeader_2.54mm:PinHeader_2x03_P2.54mm_Vertical
- +5V: value Conn_02x03_Odd_Even -> (none); footprint Connector_PinHeader_2.00mm:PinHeader_2x03_P2.00mm_Vertical -> Connector_PinHeader_2.54mm:PinHeader_2x03_P2.54mm_Vertical
- ? (x4): value MountingHole_Pad -> (none)
- C1: renamed from ?; value 100nF -> GRM21BR71E104KA01
- C2: renamed from ?; value 10uF -> GRM21BR71A106KE51
- C3: renamed from ?; value 10uF -> GRM21BR71A106KE5
- moved ? 10.2 mm to (111.8, 104.1)
- moved ? 10.2 mm to (121.9, 104.1)
- moved +5V 9.93 mm to (116.8, 97.8)
- moved C2 9.09 mm to (121.7, 92.1), turned to 0 degrees
- moved +3.3V 5.60 mm to (111.8, 86.4)
- moved L1 5.09 mm to (116.8, 88.3)
- moved C3 4.70 mm to (116.1, 83.6)
- moved C1 4.23 mm to (115.6, 79.8)
- gave numbers to parts that had none: 1
Routing:
- net GND: track 43.7 -> 19.9 mm, vias 13 -> 23
- net Net-(C2-Pad1): track 9.54 -> 13.5 mm
- net Net-(C4-Pad1): track 10.1 -> 13.5 mm
- net Net-(IC1-Pad10): track 5.29 -> 6.32 mm
- net Net-(C1-Pad1): track 30.2 -> 30.0 mm, vias 4 -> 2
Other:
- board size 19.8 x 40.1 mm -> 19.8 x 50.3 mm
- net class POWER_ added: clearance 0.2, trace_width 0.5, via_dia 0.8, via_drill 0.4
- board text added: "C2"
- board text added: "L1"
- board text added: "L2"
- board text added: "Sym. pow. supply"
- board text added: "U1"
