File: TPS65133/TPS65133_2.sch (KiCad schematic (older format))
At the start: 14 parts, among them IC1 TPS65133DPDR, J1 Conn_02x03_Odd_Even, J2 Conn_02x03_Odd_Even, J3 Conn_02x03_Odd_Even

Commit message: Update
Parts:
- added C5, C6: GRM21BR71E104KA01, Capacitor_SMD:C_0805_2012Metric, symbol Device:C
- C1: value 100nF -> GRM21BR71E104KA01
- C2, C3, C4: value 10uF -> GRM21BR71A106KE5
Connections:
- wire segments 98 -> 108
Changed lines of the file:
@@
 P 4600 2600
 F 0 "C3" V 4350 2550 50  0000 L CNN
-F 1 "10uF" V 4450 2500 50  0000 L CNN
+F 1 "GRM21BR71A106KE5" V 4450 2500 50  0000 L CNN
 F 2 "Capacitor_SMD:C_0805_2012Metric" H 4638 2450 50  0001 C CNN
 F 3 "~" H 4600 2600 50  0001 C CNN
@@
 P 3900 3700
 F 0 "C2" H 4015 3746 50  0000 L CNN
-F 1 "10uF" H 4015 3655 50  0000 L CNN
+F 1 "GRM21BR71A106KE5" H 4015 3655 50  0000 L CNN
 F 2 "Capacitor_SMD:C_0805_2012Metric" H 3938 3550 50  0001 C CNN
 F 3 "~" H 3900 3700 50  0001 C CNN
@@
 $EndComp
 Wire Wire Line
-	3900 3850 3900 4000
+	3900 3850 3900 3900
 Wire Wire Line
 	4600 3150 3900 3150
@@
 $EndComp
 Wire Wire Line
-	3900 3150 3100 3150
+	3900 3150 3500 3150
 Wire Wire Line
 	3100 3150 3100 4150
@@
 L Device:C C4
 U 1 1 5CCAD918
-P 7850 3650
-F 0 "C4" H 7965 3696 50  0000 L CNN
-F 1 "10uF" H 7965 3605 50  0000 L CNN
-F 2 "Capacitor_SMD:C_0805_2012Metric" H 7888 3500 50  0001 C CNN
-F 3 "~" H 7850 3650 50  0001 C CNN
-	1    7850 3650
+P 7550 3650
+F 0 "C4" H 7665 3696 50  0000 L CNN
+F 1 "GRM21BR71A106KE5" H 7665 3605 50  0000 L CNN
+F 2 "Capacitor_SMD:C_0805_2012Metric" H 7588 3500 50  0001 C CNN
+F 3 "~" H 7550 3650 50  0001 C CNN
+	1    7550 3650
 	1    0    0    -1
 $EndComp
@@
 L power:GND #PWR08
 U 1 1 5CCAD946
-P 7850 4000
-F 0 "#PWR08" H 7850 3750 50  0001 C CNN
-F 1 "GND" H 7855 3827 50  0000 C CNN
-F 2 "" H 7850 4000 50  0001 C CNN
-F 3 "" H 7850 4000 50  0001 C CNN
-	1    7850 4000
-	1    0    0    -1
-$EndComp
-Wire Wire Line
-	5800 3250 7850 3250
-Wire Wire Line
-	7850 3250 7850 3500
-Wire Wire Line
-	7850 3800 7850 4000
+P 7550 4000
+F 0 "#PWR08" H 7550 3750 50  0001 C CNN
+F 1 "GND" H 7555 3827 50  0000 C CNN
+F 2 "" H 7550 4000 50  0001 C CNN
+F 3 "" H 7550 4000 50  0001 C CNN
+	1    7550 4000
+	1    0    0    -1
+$EndComp
+Wire Wire Line
+	5800 3250 7550 3250
+Wire Wire Line
+	7550 3250 7550 3500
+Wire Wire Line
+	7550 3800 7550 3900
 $Comp
 L Connector_Generic:Conn_02x03_Odd_Even J3
@@
 	-1   0    0    1
 $EndComp
-Wire Wire Line
-	7850 3250 8350 3250
-Connection ~ 7850 3250
 $Comp
 L power:GND #PWR09
@@
 P 3550 1700
 F 0 "C1" V 3298 1700 50  0000 C CNN
-F 1 "100nF" V 3389 1700 50  0000 C CNN
+F 1 "GRM21BR71E104KA01" V 3389 1700 50  0000 C CNN
 F 2 "" H 3588 1550 50  0001 C CNN
 F 3 "~" H 3550 1700 50  0001 C CNN
@@
 Wire Wire Line
 	3700 1700 6100 1700
+$Comp
+L Device:C C5
+U 1 1 5CE67F0B
+P 3500 3700
+F 0 "C5" H 3615 3746 50  0000 L CNN
+F 1 "GRM21BR71E104KA01" H 3615 3655 50  0000 L CNN
+F 2 "Capacitor_SMD:C_0805_2012Metric" H 3538 3550 50  0001 C CNN
+F 3 "~" H 3500 3700 50  0001 C CNN
+	1    3500 3700
+	1    0    0    -1
+$EndComp
+Wire Wire Line
+	3500 3150 3500 3550
+Connection ~ 3500 3150
+Wire Wire Line
+	3500 3150 3100 3150
+Wire Wire Line
+	3500 3850 3500 3900
+Wire Wire Line
+	3500 3900 3900 3900
+Connection ~ 3900 3900
+Wire Wire Line
+	3900 3900 3900 4000
+Connection ~ 7550 3250
+$Comp
+L Device:C C6
+U 1 1 5CE70361
+P 8000 3650
+F 0 "C6" H 8115 3696 50  0000 L CNN
+F 1 "GRM21BR71E104KA01" H 8115 3605 50  0000 L CNN
+F 2 "Capacitor_SMD:C_0805_2012Metric" H 8038 3500 50  0001 C CNN
+F 3 "~" H 8000 3650 50  0001 C CNN
+	1    8000 3650
+	1    0    0    -1
+$EndComp
+Wire Wire Line
+	7550 3250 8000 3250
+Wire Wire Line
+	8000 3250 8000 3500
+Connection ~ 8000 3250
+Wire Wire Line
+	8000 3250 8350 3250
+Wire Wire Line
+	8000 3800 8000 3900
+Wire Wire Line
+	8000 3900 7550 3900
+Connection ~ 7550 3900
+Wire Wire Line
+	7550 3900 7550 4000
 $EndSCHEMATC

Commit message: New components
Parts:
- C1, C5, C6: value GRM21BR71E104KA01 -> 0.1uF
- C2, C3, C4: value GRM21BR71A106KE5 -> 10uF
- J1, J2, J3: footprint Connector_PinHeader_2.00mm:PinHeader_2x03_P2.00mm_Vertical -> Connector_PinHeader_2.54mm:PinHeader_2x03_P2.54mm_Vertical
Changed lines of the file:
@@
 P 4600 2600
 F 0 "C3" V 4350 2550 50  0000 L CNN
-F 1 "GRM21BR71A106KE5" V 4450 2500 50  0000 L CNN
+F 1 "10uF" V 4450 2500 50  0000 L CNN
 F 2 "Capacitor_SMD:C_0805_2012Metric" H 4638 2450 50  0001 C CNN
 F 3 "~" H 4600 2600 50  0001 C CNN
@@
 F 0 "J1" H 1300 2567 50  0000 C CNN
 F 1 "Conn_02x03_Odd_Even" H 1300 2476 50  0000 C CNN
-F 2 "Connector_PinHeader_2.00mm:PinHeader_2x03_P2.00mm_Vertical" H 1250 2250 50  0001 C CNN
+F 2 "Connector_PinHeader_2.54mm:PinHeader_2x03_P2.54mm_Vertical" H 1250 2250 50  0001 C CNN
 F 3 "~" H 1250 2250 50  0001 C CNN
 	1    1250 2250
@@
 P 3900 3700
 F 0 "C2" H 4015 3746 50  0000 L CNN
-F 1 "GRM21BR71A106KE5" H 4015 3655 50  0000 L CNN
+F 1 "10uF" H 4000 3650 50  0000 L CNN
 F 2 "Capacitor_SMD:C_0805_2012Metric" H 3938 3550 50  0001 C CNN
 F 3 "~" H 3900 3700 50  0001 C CNN
@@
 F 0 "J2" V 3104 4580 50  0000 L CNN
 F 1 "Conn_02x03_Odd_Even" V 3195 4580 50  0000 L CNN
-F 2 "Connector_PinHeader_2.00mm:PinHeader_2x03_P2.00mm_Vertical" H 3100 4400 50  0001 C CNN
+F 2 "Connector_PinHeader_2.54mm:PinHeader_2x03_P2.54mm_Vertical" H 3100 4400 50  0001 C CNN
 F 3 "~" H 3100 4400 50  0001 C CNN
 	1    3100 4400
@@
 P 7550 3650
 F 0 "C4" H 7665 3696 50  0000 L CNN
-F 1 "GRM21BR71A106KE5" H 7665 3605 50  0000 L CNN
+F 1 "10uF" H 7665 3605 50  0000 L CNN
 F 2 "Capacitor_SMD:C_0805_2012Metric" H 7588 3500 50  0001 C CNN
 F 3 "~" H 7550 3650 50  0001 C CNN
@@
 F 0 "J3" H 8850 2925 50  0000 C CNN
 F 1 "Conn_02x03_Odd_Even" H 8850 3016 50  0000 C CNN
-F 2 "Connector_PinHeader_2.00mm:PinHeader_2x03_P2.00mm_Vertical" H 8800 3250 50  0001 C CNN
+F 2 "Connector_PinHeader_2.54mm:PinHeader_2x03_P2.54mm_Vertical" H 8800 3250 50  0001 C CNN
 F 3 "~" H 8800 3250 50  0001 C CNN
 	1    8800 3250
@@
 P 3550 1700
 F 0 "C1" V 3298 1700 50  0000 C CNN
-F 1 "GRM21BR71E104KA01" V 3389 1700 50  0000 C CNN
+F 1 "0.1uF" V 3389 1700 50  0000 C CNN
 F 2 "" H 3588 1550 50  0001 C CNN
 F 3 "~" H 3550 1700 50  0001 C CNN
@@
 P 3500 3700
 F 0 "C5" H 3615 3746 50  0000 L CNN
-F 1 "GRM21BR71E104KA01" H 3615 3655 50  0000 L CNN
+F 1 "0.1uF" H 3600 3650 50  0000 L CNN
 F 2 "Capacitor_SMD:C_0805_2012Metric" H 3538 3550 50  0001 C CNN
 F 3 "~" H 3500 3700 50  0001 C CNN
@@
 P 8000 3650
 F 0 "C6" H 8115 3696 50  0000 L CNN
-F 1 "GRM21BR71E104KA01" H 8115 3605 50  0000 L CNN
+F 1 "0.1uF" H 8115 3605 50  0000 L CNN
 F 2 "Capacitor_SMD:C_0805_2012Metric" H 8038 3500 50  0001 C CNN
 F 3 "~" H 8000 3650 50  0001 C CNN

Commit message: upravy, pred vyrobou, opraven problem s maskou
Parts:
- IC1: symbol SamacSys_Parts:TPS65133DPDR -> TPS65133_2-rescue:TPS65133DPDR-SamacSys_Parts
- L1, L2: symbol SamacSys_Parts:1239AS-H-4R7M=P2 -> TPS65133_2-rescue:1239AS-H-4R7M=P2-SamacSys_Parts
Changed lines of the file:
@@
 $EndDescr
 $Comp
-L SamacSys_Parts:TPS65133DPDR IC1
+L TPS65133_2-rescue:TPS65133DPDR-SamacSys_Parts IC1
 U 1 1 5CC9FF14
 P 4600 2950
@@
 $EndComp
 $Comp
-L SamacSys_Parts:1239AS-H-4R7M=P2 L1
+L TPS65133_2-rescue:1239AS-H-4R7M=P2-SamacSys_Parts L1
 U 1 1 5CCA0079
 P 4800 2250
@@
 $EndComp
 $Comp
-L SamacSys_Parts:1239AS-H-4R7M=P2 L2
+L TPS65133_2-rescue:1239AS-H-4R7M=P2-SamacSys_Parts L2
 U 1 1 5CCA00D1
 P 6500 3650
