File: Analog_board/Analog_board.kicad_pcb (KiCad board)
At the start: 4 copper layers, 65.5 x 134.1 mm, 85 parts, among them J1 02x03_Female, J10 01x03_Male, J11 02x04_Male, J12 01x02_Male, J13 01x03_Female, J14 01x03_Female, J2 02x03_Female, J3 02x04_Female, J4 02x03_Female, J5 02x03_Female, J6 02x03_Female, J7 02x04_Male, J8 Conn_Coaxial, J9 01x03_Male, U2 OPA656, U3 CAT5140ZI-00-GT3, U4 TMP1075, U5 LM337_SOT223, U6 MCP3021, U7 LMH6553, U8 LMH6553

Commit message: F.fab
Parts:
- IN +3.3V: renamed from J1
- renumbered J4 to +3.3V, J2 to +3.3V, J5 to +5V, J3 to -32V, J6 to -5V, J11 to Alert_tem, R34 to High, J9 to JP, R33 to Low, J12 to Ohm_meter, R1 to SCL, R2 to SDA, J13 to SiPM_IN, J14 to SiPM_OUT, J10 to Volt_meter, R3 to WP
Other:
- board text added: "DIGI_POT"
- board text added: "RESISTOR"

Commit message: New components
Parts:
- High, Low, R13, R14, R31, R32, R35: value 50R -> 49.9R
- R10: value 120R -> 121R
- R11, R29, R30: value 4k -> 4.02k
- R12: value 26k -> 26.1k
- R27, R28: value 500R -> 499R
- R7: value 470R -> 464R
- R8: value 30k -> 30.1k
- R9: value 2.7k -> 2.67k
Changed lines of the file:
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@@
       (effects (font (size 1 1) (thickness 0.15)))
     )
-    (fp_text value 470R (at 0 -1.778 180) (layer F.Fab) hide
+    (fp_text value 464R (at 0 -1.778 180) (layer F.Fab) hide
       (effects (font (size 1 1) (thickness 0.15)))
     )
@@
       (effects (font (size 1 1) (thickness 0.15)))
     )
-    (fp_text value 30k (at 0.254 -1.6764) (layer F.Fab) hide
+    (fp_text value 30.1k (at 0.254 -1.6764) (layer F.Fab) hide
       (effects (font (size 1 1) (thickness 0.15)))
     )
@@
       (effects (font (size 1 1) (thickness 0.15)))
     )
-    (fp_text value 2.7k (at -0.1016 -1.5748 180) (layer F.Fab) hide
+    (fp_text value 2.67k (at -0.1016 -1.5748 180) (layer F.Fab) hide
       (effects (font (size 1 1) (thickness 0.15)))
     )
@@
       (effects (font (size 1 1) (thickness 0.15)))
     )
-    (fp_text value 120R (at 0.127 1.5748 180) (layer F.Fab) hide
+    (fp_text value 121R (at 0.127 1.5748 180) (layer F.Fab) hide
       (effects (font (size 1 1) (thickness 0.15)))
     )
@@
       (effects (font (size 1 1) (thickness 0.15)))
     )
-    (fp_text value 4k (at 0 1.65 90) (layer F.Fab) hide
+    (fp_text value 4.02k (at 0 1.65 90) (layer F.Fab) hide
       (effects (font (size 1 1) (thickness 0.15)))
     )
@@
       (effects (font (size 1 1) (thickness 0.15)))
     )
-    (fp_text value 26k (at 0 1.65 180) (layer F.Fab) hide
+    (fp_text value 26.1k (at 0 1.65 180) (layer F.Fab) hide
       (effects (font (size 1 1) (thickness 0.15)))
     )
@@
       (effects (font (size 1 1) (thickness 0.15)))
     )
-    (fp_text value 50R (at 0 -1.778 270) (layer F.Fab) hide
+    (fp_text value 49.9R (at 0 -1.778 270) (layer F.Fab) hide
       (effects (font (size 1 1) (thickness 0.15)))
     )
@@
       (effects (font (size 1 1) (thickness 0.15)))
     )
-    (fp_text value 50R (at -0.0785 -1.778 270) (layer F.Fab) hide
+    (fp_text value 49.9R (at -0.0785 -1.778 270) (layer F.Fab) hide
       (effects (font (size 1 1) (thickness 0.15)))
     )
@@
       (effects (font (size 1 1) (thickness 0.15)))
     )
-    (fp_text value 500R (at -0.0785 1.778) (layer F.Fab) hide
+    (fp_text value 499R (at -0.0785 1.778) (layer F.Fab) hide
       (effects (font (size 1 1) (thickness 0.15)))
     )
@@
       (effects (font (size 1 1) (thickness 0.15)))
     )
-    (fp_text value 500R (at -0.508 1.524 270) (layer F.Fab) hide
+    (fp_text value 499R (at -0.508 1.524 270) (layer F.Fab) hide
       (effects (font (size 1 1) (thickness 0.15)))
     )
@@
       (effects (font (size 1 1) (thickness 0.15)))
     )
-    (fp_text value 4k (at 0 1.65 90) (layer F.Fab) hide
+    (fp_text value 4.02k (at 0 1.65 90) (layer F.Fab) hide
       (effects (font (size 1 1) (thickness 0.15)))
     )
@@
       (effects (font (size 1 1) (thickness 0.15)))
     )
-    (fp_text value 4k (at 0 1.65 90) (layer F.Fab) hide
+    (fp_text value 4.02k (at 0 1.65 90) (layer F.Fab) hide
       (effects (font (size 1 1) (thickness 0.15)))
     )
@@
       (effects (font (size 1 1) (thickness 0.15)))
     )
-    (fp_text value 50R (at 0.03326 -1.6764) (layer F.Fab) hide
+    (fp_text value 49.9R (at 0.03326 -1.6764) (layer F.Fab) hide
       (effects (font (size 1 1) (thickness 0.15)))
     )
@@
       (effects (font (size 1 1) (thickness 0.15)))
     )
-    (fp_text value 50R (at 0 1.65 180) (layer F.Fab) hide
+    (fp_text value 49.9R (at 0 1.65 180) (layer F.Fab) hide
       (effects (font (size 1 1) (thickness 0.15)))
     )
@@
       (effects (font (size 1 1) (thickness 0.15)))
     )
-    (fp_text value 50R (at -0.1755 -1.524) (layer F.Fab) hide
+    (fp_text value 49.9R (at -0.1755 -1.524) (layer F.Fab) hide
       (effects (font (size 1 1) (thickness 0.15)))
     )
@@
       (effects (font (size 1 1) (thickness 0.15)))
     )
-    (fp_text value 50R (at 0 1.65) (layer F.Fab) hide
+    (fp_text value 49.9R (at 0 1.65) (layer F.Fab) hide
       (effects (font (size 1 1) (thickness 0.15)))
     )
@@
       (effects (font (size 1 1) (thickness 0.15)))
     )
-    (fp_text value 50R (at 0 -2.032 180) (layer F.Fab) hide
-      (effects (font (size 1 1) (thickness 0.15)))
-    )
+    (fp_text value 49.9R (at 0 -2.032 180) (layer F.Fab) hide
+      (effects (font (size 1 1) (thickness 0.15)))
+    )
