File: Analog_board/Diff_amp.sch (KiCad schematic (older format))
At the start: 33 parts, among them U7 LMH6553, U8 LMH6553

Commit message: New components
Parts:
- R13, R14, R31, R32, R33, R34, R35: value 50R -> 49.9R
- R27, R28: value 500R -> 499R
- R29, R30: value 4k -> 4.02k
Changed lines of the file:
@@
 P 1400 3100
 F 0 "R13" H 1470 3146 50  0000 L CNN
-F 1 "50R" H 1470 3055 50  0000 L CNN
+F 1 "49.9R" H 1470 3055 50  0000 L CNN
 F 2 "Resistor_SMD:R_0805_2012Metric" V 1330 3100 50  0001 C CNN
 F 3 "~" H 1400 3100 50  0001 C CNN
@@
 P 3500 5400
 F 0 "R27" V 3293 5400 50  0000 C CNN
-F 1 "500R" V 3384 5400 50  0000 C CNN
+F 1 "499R" V 3384 5400 50  0000 C CNN
 F 2 "Resistor_SMD:R_0805_2012Metric" V 3430 5400 50  0001 C CNN
 F 3 "~" H 3500 5400 50  0001 C CNN
@@
 P 3500 6950
 F 0 "R28" V 3293 6950 50  0000 C CNN
-F 1 "500R" V 3384 6950 50  0000 C CNN
+F 1 "499R" V 3384 6950 50  0000 C CNN
 F 2 "Resistor_SMD:R_0805_2012Metric" V 3430 6950 50  0001 C CNN
 F 3 "~" H 3500 6950 50  0001 C CNN
@@
 P 3850 1600
 F 0 "R29" V 4057 1600 50  0000 C CNN
-F 1 "4k" V 3966 1600 50  0000 C CNN
+F 1 "4.02k" V 3966 1600 50  0000 C CNN
 F 2 "Resistor_SMD:R_0805_2012Metric" V 3780 1600 50  0001 C CNN
 F 3 "~" H 3850 1600 50  0001 C CNN
@@
 P 3850 5550
 F 0 "R30" V 4057 5550 50  0000 C CNN
-F 1 "4k" V 3966 5550 50  0000 C CNN
+F 1 "4.02k" V 3966 5550 50  0000 C CNN
 F 2 "Resistor_SMD:R_0805_2012Metric" V 3780 5550 50  0001 C CNN
 F 3 "~" H 3850 5550 50  0001 C CNN
@@
 P 1400 5250
 F 0 "R14" H 1470 5296 50  0000 L CNN
-F 1 "50R" H 1470 5205 50  0000 L CNN
+F 1 "49.9R" H 1470 5205 50  0000 L CNN
 F 2 "Resistor_SMD:R_0805_2012Metric" V 1330 5250 50  0001 C CNN
 F 3 "~" H 1400 5250 50  0001 C CNN
@@
 AR Path="/5C99A3DD/5C9D9D19" Ref="R32"  Part="1"
 F 0 "R32" V 5843 2000 50  0000 C CNN
-F 1 "50R" V 5934 2000 50  0000 C CNN
+F 1 "49.9R" V 5934 2000 50  0000 C CNN
 F 2 "Resistor_SMD:R_0805_2012Metric" V 5980 2000 50  0001 C CNN
 F 3 "~" H 6050 2000 50  0001 C CNN
@@
 AR Path="/5C99A3DD/5C9D9D27" Ref="R33"  Part="1"
 F 0 "R33" V 5843 2400 50  0000 C CNN
-F 1 "50R" V 5934 2400 50  0000 C CNN
+F 1 "49.9R" V 5934 2400 50  0000 C CNN
 F 2 "Resistor_SMD:R_0805_2012Metric" V 5980 2400 50  0001 C CNN
 F 3 "~" H 6050 2400 50  0001 C CNN
@@
 AR Path="/5C99A3DD/5C9E420B" Ref="R34"  Part="1"
 F 0 "R34" V 5843 5950 50  0000 C CNN
-F 1 "50R" V 5934 5950 50  0000 C CNN
+F 1 "49.9R" V 5934 5950 50  0000 C CNN
 F 2 "Resistor_SMD:R_0805_2012Metric" V 5980 5950 50  0001 C CNN
 F 3 "~" H 6050 5950 50  0001 C CNN
@@
 AR Path="/5C99A3DD/5C9E4219" Ref="R35"  Part="1"
 F 0 "R35" V 5843 6350 50  0000 C CNN
-F 1 "50R" V 5934 6350 50  0000 C CNN
+F 1 "49.9R" V 5934 6350 50  0000 C CNN
 F 2 "Resistor_SMD:R_0805_2012Metric" V 5980 6350 50  0001 C CNN
 F 3 "~" H 6050 6350 50  0001 C CNN
@@
 P 5900 4200
 F 0 "R31" V 5693 4200 50  0000 C CNN
-F 1 "50R" V 5784 4200 50  0000 C CNN
+F 1 "49.9R" V 5784 4200 50  0000 C CNN
 F 2 "Resistor_SMD:R_0805_2012Metric" V 5830 4200 50  0001 C CNN
 F 3 "~" H 5900 4200 50  0001 C CNN
