File: Analog_board/Power_regulation.sch (KiCad schematic (older format))
At the start: 18 parts, among them J10 Conn_01x03_Male, J12 Conn_01x02_Male, J9 Conn_01x03_Male, U3 CAT5140ZI-00-GT3, U4 TMP1075, U5 LM337_SOT223, U6 MCP3021

Commit message: New components
Parts:
- R10: value 120R -> 121R
- R11: value 4k -> 4.02k
- R12: value 26k -> 26.1k
- R8: value 30k -> 30.1k
- R9: value 2.7k -> 2.67k
Changed lines of the file:
@@
 P 6700 3400
 F 0 "R12" H 6770 3446 50  0000 L CNN
-F 1 "26k" H 6770 3355 50  0000 L CNN
+F 1 "26.1k" H 6770 3355 50  0000 L CNN
 F 2 "Resistor_SMD:R_0805_2012Metric" V 6630 3400 50  0001 C CNN
 F 3 "~" H 6700 3400 50  0001 C CNN
@@
 P 6700 1950
 F 0 "R11" H 6770 1996 50  0000 L CNN
-F 1 "4k" H 6770 1905 50  0000 L CNN
+F 1 "4.02k" H 6770 1905 50  0000 L CNN
 F 2 "Resistor_SMD:R_0805_2012Metric" V 6630 1950 50  0001 C CNN
 F 3 "~" H 6700 1950 50  0001 C CNN
@@
 P 5150 3750
 F 0 "R10" H 5220 3796 50  0000 L CNN
-F 1 "120R" H 5220 3705 50  0000 L CNN
+F 1 "121R" H 5220 3705 50  0000 L CNN
 F 2 "Resistor_SMD:R_0805_2012Metric" V 5080 3750 50  0001 C CNN
 F 3 "~" H 5150 3750 50  0001 C CNN
@@
 P 4650 2100
 F 0 "R9" H 4720 2146 50  0000 L CNN
-F 1 "2.7k" H 4720 2055 50  0000 L CNN
+F 1 "2.67k" H 4720 2055 50  0000 L CNN
 F 2 "Resistor_SMD:R_0805_2012Metric" V 4580 2100 50  0001 C CNN
 F 3 "~" H 4650 2100 50  0001 C CNN
@@
 P 4250 2450
 F 0 "R8" V 4043 2450 50  0000 C CNN
-F 1 "30k" V 4134 2450 50  0000 C CNN
+F 1 "30.1k" V 4134 2450 50  0000 C CNN
 F 2 "Resistor_SMD:R_0805_2012Metric" V 4180 2450 50  0001 C CNN
 F 3 "~" H 4250 2450 50  0001 C CNN
