File: Analog_board/SiPM_TIA.sch (KiCad schematic (older format))
At the start: 18 parts, among them J13 Conn_01x03_Female, J14 Conn_01x03_Female, U2 OPA656

Commit message: New components
Parts:
- R7: value 470R -> 464R
Changed lines of the file:
@@
 AR Path="/5C966022/5C969A53" Ref="R7"  Part="1"
 F 0 "R7" V 7393 4400 50  0000 C CNN
-F 1 "470R" V 7484 4400 50  0000 C CNN
+F 1 "464R" V 7484 4400 50  0000 C CNN
 F 2 "Resistor_SMD:R_0805_2012Metric" V 7530 4400 50  0001 C CNN
 F 3 "~" H 7600 4400 50  0001 C CNN
